File: PCB Files/406MHz detector/406MHz detector.sch (EAGLE design)
At the start: 35 parts, among them J1 switch, J3 select jumper, U2 ATMEGA328P_TQFP, Y1 8MHz

Commit message: added ftdi adaptor, small schematic changes
Parts:
- added C13: 2.2uF, SparkFun-Capacitors:2.2UF-0805-25V-(+80/-20%)
- added IC1: FT232RL, ftdichip:FT232RL
- added J4: select jumper, SparkFun-Connectors:CONN_03LOCK
- added J5: reset switch, SparkFun-Connectors:CONN_02
- added J6: (no value), SparkFun-Connectors:CONN_02
- added JP1, JP2, JP3, JP4: JUMPER-SMT_2_NO_SILK_ROUND, SparkFun-Jumpers:JUMPER-SMT_2_NO_SILK_ROUND
- added JP5: JUMPER-SMT_3_NO_SILK, SparkFun-Jumpers:JUMPER-SMT_3_NO_SILK
- added JP6: JUMPER-SMT_3_2-NC_TRACE_SILK, SparkFun-Jumpers:JUMPER-SMT_3_2-NC_TRACE_SILK
- added R10: 100K, SparkFun-Resistors:100KOHM-0402-1/16W-1%
- added R7, R8: 100, SparkFun-Resistors:100KOHM-0402-1/16W-1%
- added TP1, TP2: TEST-POINT3X5, SparkFun-Connectors:TEST-POINT3X5
- J1: value switch -> power switch
- J2: value (none) -> pwr_input
- R3, R4: value 10k -> 100; device SparkFun-Resistors:10KOHM-0603-1/10W-1% -> SparkFun-Resistors:100KOHM-0402-1/16W-1%
- R5, R6: value 150 -> 100; device SparkFun-Resistors:150OHM-0603-1/10W-1% -> SparkFun-Resistors:100KOHM-0402-1/16W-1%
Connections:
- net N$10 renamed CSRM_OSC_OUT
- net N$11 renamed CSRM_GPIO1
- net N$12 renamed CSRM_GPIO2
- net N$13 renamed CSRM_GPIO3
- net N$9 renamed !CSRM_LED_SINK
- removed net N$18: J3.1
- removed net N$19: J3.2
- removed net N$20: J3.3
- removed net N$23: R3.1
- removed net N$24: R4.1
- removed net N$25: R6.1
- removed net N$26: R5.1
- removed net RESET_UC: R9.1, U2.PC6(/RESET)
- new net CSRM_EN: R8.1, U$3.EN
- new net CSRM_PPS: R3.2, U2.PB0(ICP)
- new net CSRM_RESET: JP6.1, U$3.RESET
- new net CSRM_RX: J4.2, JP3.1, R6.1
- new net CSRM_TX: J3.2, JP4.1, R7.1
- new net EJECT_SD: J6.2
- new net GPS_SERIAL_IN: JP2.1, R5.1
- new net GPS_SERIAL_OUT: JP1.1, R4.1
- new net MOSI: U2.PB3(MOSI/OC2)
- new net MSIO: U2.PB4(MISO)
- new net N$10: R10.1
- new net N$12: IC1.VCCIO
- new net N$13: IC1.USBDP
- new net N$9: IC1.!RESET, R10.2
- new net RESET: C13.1, J5.2, JP6.2
- new net SCLK: U2.PB5(SCK)
- new net SS: U2.PB2(SS/OC1B)
- new net UC_RESET: JP6.3, R9.1, U2.PC6(/RESET)
- new net UC_RX: J3.1, U2.PD0(RXD)
- new net UC_TX: J4.1, U2.PD1(TXD)
- new net USB_RX: IC1.RXD, J3.3, TP2.1
- new net USB_TX: IC1.TXD, J4.3, TP1.1
- new net USB_VCC: IC1.VCC
- net 3.3V: now also JP5.1; no longer R3.2, R4.2, R5.2, R6.2
- net GND: now also C13.2, IC1.GND, IC1.GND@1, IC1.GND@2, IC1.GND@A, J5.1, J6.1, JP5.3
- net N$1: now also JP1.2, R4.2, U$3.TX1; no longer U$3.EN
- net N$14: now also IC1.USBDM; no longer U$3.RESET
- net N$3: now also R3.1, U$3.PPS; no longer U$3.TX1
- net N$4: now also JP2.2, R5.2
- net N$5: now also JP3.2, R6.2
- net N$6: now also JP4.2, R7.2
- net N$8: now also JP5.2, R8.2; no longer U$3.PPS
Other:
- moved on the sheet: C11, C12, C6, J3, L2, L3, R3, R4, R5, R6, R9, U$3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

Commit message: small changes to PCB
Parts:
- added C14: 10uF, SparkFun-Capacitors:10UF-1206-6.3V-20%
Connections:
- removed net N$10: R10.1
- removed net N$12: IC1.VCCIO
- net 3.3V: now also C14.1, IC1.3V3OUT, IC1.VCCIO
- net GND: now also C14.2
- net UC_RESET: now also R10.1
Changed lines of the file:
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@@
 <part name="TP1" library="SparkFun-Connectors" library_urn="urn:adsk.eagle:library:513" deviceset="TEST-POINT" device="3X5" package3d_urn="urn:adsk.eagle:package:38285/1"/>
 <part name="TP2" library="SparkFun-Connectors" library_urn="urn:adsk.eagle:library:513" deviceset="TEST-POINT" device="3X5" package3d_urn="urn:adsk.eagle:package:38285/1"/>
+<part name="C14" library="SparkFun-Capacitors" library_urn="urn:adsk.eagle:library:510" deviceset="10UF" device="-1206-6.3V-20%" package3d_urn="urn:adsk.eagle:package:37426/1" value="10uF"/>
 </parts>
 <sheets>
@@
 <attribute name="VALUE" x="307.34" y="175.26" size="1.778" layer="96" font="vector"/>
 </instance>
+<instance part="C14" gate="G$1" x="233.68" y="154.94" smashed="yes">
+<attribute name="NAME" x="235.204" y="157.861" size="1.778" layer="95" font="vector"/>
+<attribute name="VALUE" x="235.204" y="152.781" size="1.778" layer="96" font="vector"/>
+</instance>
 </instances>
 <busses>
@@
 <wire x1="416.56" y1="78.74" x2="414.02" y2="78.74" width="0.1524" layer="91"/>
 <label x="414.02" y="78.74" size="1.27" layer="95" rot="R180" xref="yes"/>
+</segment>
+<segment>
+<pinref part="IC1" gate="1" pin="VCCIO"/>
+<wire x1="261.62" y1="185.42" x2="233.68" y2="185.42" width="0.1524" layer="91"/>
+<wire x1="233.68" y1="185.42" x2="233.68" y2="160.02" width="0.1524" layer="91"/>
+<pinref part="IC1" gate="1" pin="3V3OUT"/>
+<wire x1="233.68" y1="160.02" x2="261.62" y2="160.02" width="0.1524" layer="91"/>
+<pinref part="C14" gate="G$1" pin="1"/>
+<junction x="233.68" y="160.02"/>
 </segment>
 </net>
@@
 <wire x1="261.62" y1="134.62" x2="289.56" y2="134.62" width="0.1524" layer="91"/>
 <junction x="289.56" y="134.62"/>
+<pinref part="C14" gate="G$1" pin="2"/>
+<wire x1="233.68" y1="152.4" x2="233.68" y2="134.62" width="0.1524" layer="91"/>
+<wire x1="233.68" y1="134.62" x2="261.62" y2="134.62" width="0.1524" layer="91"/>
+<junction x="261.62" y="134.62"/>
 </segment>
 </net>
@@
 <label x="200.66" y="45.72" size="1.27" layer="95" xref="yes"/>
 </segment>
+<segment>
+<pinref part="R10" gate="G$1" pin="1"/>
+<wire x1="243.84" y1="180.34" x2="238.76" y2="180.34" width="0.1524" layer="91"/>
+<label x="238.76" y="180.34" size="1.27" layer="95" rot="R180" xref="yes"/>
+</segment>
 </net>
 <net name="CSRM_RESET" class="0">
@@
 </segment>
 </net>
-<net name="N$10" class="0">
-<segment>
-<pinref part="R10" gate="G$1" pin="1"/>
-<wire x1="243.84" y1="180.34" x2="238.76" y2="180.34" width="0.1524" layer="91"/>
-</segment>
-</net>
 <net name="USB_VCC" class="0">
 <segment>
@@
 </segment>
 </net>
-<net name="N$12" class="0">
-<segment>
-<pinref part="IC1" gate="1" pin="VCCIO"/>
-<wire x1="261.62" y1="185.42" x2="238.76" y2="185.42" width="0.1524" layer="91"/>
-</segment>
-</net>

Commit message: added labels to usb pins
Connections:
- net N$13 renamed USB_DP
- net N$14 renamed USB_DM
Changed lines of the file:
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@@
 </segment>
 </net>
-<net name="N$13" class="0">
+<net name="USB_DP" class="0">
 <segment>
 <pinref part="IC1" gate="1" pin="USBDP"/>
 <wire x1="261.62" y1="154.94" x2="256.54" y2="154.94" width="0.1524" layer="91"/>
+<label x="256.54" y="154.94" size="1.27" layer="95" rot="R180" xref="yes"/>
 </segment>
 </net>
-<net name="N$14" class="0">
+<net name="USB_DM" class="0">
 <segment>
 <pinref part="IC1" gate="1" pin="USBDM"/>
 <wire x1="261.62" y1="152.4" x2="256.54" y2="152.4" width="0.1524" layer="91"/>
+<label x="256.54" y="152.4" size="1.27" layer="95" rot="R180" xref="yes"/>
 </segment>
 </net>

Commit message: removed old footprints from library, added usb connector
Parts:
- added C15, C16, C17: 0.18uF, SparkFun-Capacitors:0.18UF-0603-10V-10%
- added U$1: USB-B, capstone:USB-B
Connections:
- net ANTENNA renamed ANTENNA_CONNECTOR
- net 3.3V: now also C15.1, C17.1
- net GND: now also C15.2, C16.2, C17.2
- net USB_VCC: now also C16.1
Changed lines of the file:
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@@
 <part name="TP2" library="SparkFun-Connectors" library_urn="urn:adsk.eagle:library:513" deviceset="TEST-POINT" device="3X5" package3d_urn="urn:adsk.eagle:package:38285/1"/>
 <part name="C14" library="SparkFun-Capacitors" library_urn="urn:adsk.eagle:library:510" deviceset="10UF" device="-1206-6.3V-20%" package3d_urn="urn:adsk.eagle:package:37426/1" value="10uF"/>
+<part name="C15" library="SparkFun-Capacitors" library_urn="urn:adsk.eagle:library:510" deviceset="0.18UF" device="-0603-10V-10%" package3d_urn="urn:adsk.eagle:package:37414/1" value="0.18uF"/>
+<part name="GND19" library="SparkFun-PowerSymbols" library_urn="urn:adsk.eagle:library:530" deviceset="GND" device=""/>
+<part name="C16" library="SparkFun-Capacitors" library_urn="urn:adsk.eagle:library:510" deviceset="0.18UF" device="-0603-10V-10%" package3d_urn="urn:adsk.eagle:package:37414/1" value="0.18uF"/>
+<part name="GND20" library="SparkFun-PowerSymbols" library_urn="urn:adsk.eagle:library:530" deviceset="GND" device=""/>
+<part name="C17" library="SparkFun-Capacitors" library_urn="urn:adsk.eagle:library:510" deviceset="0.18UF" device="-0603-10V-10%" package3d_urn="urn:adsk.eagle:package:37414/1" value="0.18uF"/>
+<part name="GND21" library="SparkFun-PowerSymbols" library_urn="urn:adsk.eagle:library:530" deviceset="GND" device=""/>
+<part name="U$1" library="capstone" deviceset="USB-B" device=""/>
 </parts>
 <sheets>
@@
 <attribute name="VALUE" x="235.204" y="152.781" size="1.778" layer="96" font="vector"/>
 </instance>
+<instance part="C15" gate="G$1" x="243.84" y="86.36" smashed="yes">
+<attribute name="NAME" x="245.364" y="89.281" size="1.778" layer="95" font="vector"/>
+<attribute name="VALUE" x="245.364" y="84.201" size="1.778" layer="96" font="vector"/>
+</instance>
+<instance part="GND19" gate="1" x="243.84" y="81.28" smashed="yes">
+<attribute name="VALUE" x="243.84" y="81.026" size="1.778" layer="96" align="top-center"/>
+</instance>
+<instance part="C16" gate="G$1" x="246.38" y="198.12" smashed="yes">
+<attribute name="NAME" x="247.904" y="201.041" size="1.778" layer="95" font="vector"/>
+<attribute name="VALUE" x="247.904" y="195.961" size="1.778" layer="96" font="vector"/>
+</instance>
+<instance part="GND20" gate="1" x="246.38" y="190.5" smashed="yes">
+<attribute name="VALUE" x="246.38" y="190.246" size="1.778" layer="96" align="top-center"/>
+</instance>
+<instance part="C17" gate="G$1" x="109.22" y="86.36" smashed="yes">
+<attribute name="NAME" x="110.744" y="89.281" size="1.778" layer="95" font="vector"/>
+<attribute name="VALUE" x="110.744" y="84.201" size="1.778" layer="96" font="vector"/>
+</instance>
+<instance part="GND21" gate="1" x="109.22" y="78.74" smashed="yes">
+<attribute name="VALUE" x="109.22" y="78.486" size="1.778" layer="96" align="top-center"/>
+</instance>
+<instance part="U$1" gate="G$1" x="119.38" y="297.18" smashed="yes">
+<attribute name="NAME" x="114.3" y="305.054" size="1.778" layer="95" font="vector"/>
+<attribute name="VALUE" x="114.3" y="291.846" size="1.778" layer="96" font="vector" align="top-left"/>
+</instance>
 </instances>
 <busses>
@@
 <segment>
 <pinref part="U$3" gate="G$1" pin="3.3V+"/>
-<wire x1="116.84" y1="78.74" x2="111.76" y2="78.74" width="0.1524" layer="91"/>
-<label x="111.76" y="78.74" size="1.27" layer="95" rot="R180" xref="yes"/>
+<wire x1="116.84" y1="78.74" x2="116.84" y2="93.98" width="0.1524" layer="91"/>
+<wire x1="116.84" y1="93.98" x2="109.22" y2="93.98" width="0.1524" layer="91"/>
+<wire x1="109.22" y1="91.44" x2="109.22" y2="93.98" width="0.1524" layer="91"/>
+<wire x1="109.22" y1="93.98" x2="106.68" y2="93.98" width="0.1524" layer="91"/>
+<label x="106.68" y="93.98" size="1.27" layer="95" rot="R180" xref="yes"/>
+<pinref part="C17" gate="G$1" pin="1"/>
+<junction x="109.22" y="93.98"/>
 </segment>
 <segment>
@@
 <wire x1="251.46" y1="91.44" x2="251.46" y2="88.9" width="0.1524" layer="91"/>
 <junction x="251.46" y="91.44"/>
-<wire x1="251.46" y1="91.44" x2="241.3" y2="91.44" width="0.1524" layer="91"/>
+<wire x1="251.46" y1="91.44" x2="243.84" y2="91.44" width="0.1524" layer="91"/>
 <label x="241.3" y="91.44" size="1.27" layer="95" rot="R180" xref="yes"/>
 <pinref part="U2" gate="U$1" pin="AREF"/>
+<wire x1="243.84" y1="91.44" x2="241.3" y2="91.44" width="0.1524" layer="91"/>
 <wire x1="251.46" y1="83.82" x2="251.46" y2="88.9" width="0.1524" layer="91"/>
 <junction x="251.46" y="88.9"/>
+<pinref part="C15" gate="G$1" pin="1"/>
+<junction x="243.84" y="91.44"/>
 </segment>
 <segment>
@@
 <junction x="261.62" y="134.62"/>
 </segment>
+<segment>
+<pinref part="C15" gate="G$1" pin="2"/>
+<pinref part="GND19" gate="1" pin="GND"/>
+</segment>
+<segment>
+<pinref part="C16" gate="G$1" pin="2"/>
+<pinref part="GND20" gate="1" pin="GND"/>
+<wire x1="246.38" y1="195.58" x2="246.38" y2="193.04" width="0.1524" layer="91"/>
+</segment>
+<segment>
+<pinref part="C17" gate="G$1" pin="2"/>
+<pinref part="GND21" gate="1" pin="GND"/>
+<wire x1="109.22" y1="83.82" x2="109.22" y2="81.28" width="0.1524" layer="91"/>
+</segment>
 </net>
 <net name="CSRM_EN" class="0">
@@
 </segment>
 </net>
-<net name="ANTENNA" class="0">
+<net name="ANTENNA_CONNECTOR" class="0">
 <segment>
 <pinref part="C6" gate="G$1" pin="1"/>
@@
 <segment>
 <pinref part="IC1" gate="1" pin="VCC"/>
-<wire x1="261.62" y1="187.96" x2="238.76" y2="187.96" width="0.1524" layer="91"/>
-<label x="238.76" y="187.96" size="1.27" layer="95" rot="R180" xref="yes"/>
-</segment>
-</net>
+<wire x1="261.62" y1="187.96" x2="256.54" y2="187.96" width="0.1524" layer="91"/>
+<wire x1="256.54" y1="187.96" x2="256.54" y2="203.2" width="0.1524" layer="91"/>
+<wire x1="256.54" y1="203.2" x2="246.38" y2="203.2" width="0.1524" layer="91"/>
+<wire x1="246.38" y1="203.2" x2="238.76" y2="203.2" width="0.1524" layer="91"/>
+<label x="238.76" y="203.2" size="1.27" layer="95" rot="R180" xref="yes"/>
+<pinref part="C16" gate="G$1" pin="1"/>
+<junction x="246.38" y="203.2"/>
+</segment>
+</net>

Commit message: added gps module to schematic
Parts:
- added C18: 0.1uF, SparkFun-Capacitors:0.18UF-0603-10V-10%
- added R11: 100K, SparkFun-Resistors:100KOHM-0402-1/16W-1%
- added U$6: WST_GPS, capstone:WST_GPS
- C13, C7: value 2.2uF -> 0.1uF
- C15, C16, C17: value 0.18uF -> 0.1uF
Connections:
- new net GPS_ANTENNA: U$6.RF_IN
- new net GPS_ENABLE: R11.1, U$6.ON_OFF
- new net N$11: U$6.V_BAT
- new net N$12: U$6.WAKE
- new net N$14: U$6.I2C_DIO
- new net N$18: U$6.I2C_CLK
- new net N$19: U$6.BOOTSEL
- new net N$23: U$6.RESET
- new net N$24: U$6.PPS
- new net N$25: U$6.RX
- new net N$26: U$6.TX
- net 3.3V: now also C18.1, R11.2, U$6.VCC
- net GND: now also C18.2, U$6.GND
Other:
- moved on the sheet: U$1

Commit message: latest version of sch and brd
Parts:
- removed JP5: JUMPER-SMT_3_NO_SILK, SparkFun-Jumpers:JUMPER-SMT_3_NO_SILK
- added C19: TBD, SparkFun-Capacitors:0.1UF-0603-25V-5%
- added C20: 0.1uF, SparkFun-Capacitors:0.18UF-0603-10V-10%
- added JP7: card detect, SparkFun-Jumpers:JUMPER-SMT_2_NO_SILK
- added L7, L8: TBD, SparkFun-Coils:INDUCTOR-0603-33NH
- added R12: 10k, SparkFun-Resistors:10KOHM-0603-1/10W-1%
- added U$7: A32270-ND, capstone:A32270-ND
- added U$8: SD_CARD_HOLDER, capstone:SD_CARD_HOLDER
- C6: value 0.1uF -> TBD
- L2, L3: value 33nH/±5%/500mA -> TBD
Connections:
- removed net MSIO: U2.PB4(MISO)
- new net GPS_CONNECTOR: C19.1, L8.1
- new net MISO: U$8.DAT0, U2.PB4(MISO)
- new net N$10: IC1.CBUS0
- new net N$13: JP7.1, U$8.CD/DAT3
- new net N$27: U2.PD6(AIN0)
- new net SD_CD: JP7.2, R12.1, U2.PD7(AIN1)
- net 3.3V: now also C20.1, R12.2, U$8.VDD; no longer JP5.1
- net ANTENNA_CONNECTOR: now also U$7.OUT
- net CSRM_EN: no longer U$3.EN
- net GND: now also C20.2, L7.2, L8.2, U$1.GND, U$1.SHIELD, U$7.GND, U$8.VSS; no longer JP5.3
- net GPS_ANTENNA: now also C19.2, L7.1
- net MOSI: now also U$8.CMD
- net N$8: now also U$3.EN; no longer JP5.2
- net SCLK: now also U$8.CLK
- net USB_DM: now also U$1.D-
- net USB_DP: now also U$1.D+
- net USB_VCC: now also U$1.VBUS
Other:
- moved on the sheet: R8, U$1

Commit message: ensuring updates are pushed
Parts:
- removed JP7: card detect, SparkFun-Jumpers:JUMPER-SMT_2_NO_SILK
- removed U$1: USB-B, capstone:USB-B
- removed U$3: CSRM100, capstone:CSRM100
- removed U$5: DIODE, capstone:DIODE
- removed U$7: A32270-ND, capstone:A32270-ND
- added C21: 0.1uF, SparkFun-Capacitors:0.18UF-0603-10V-10%
- added C22: TBD, SparkFun-Capacitors:0.1UF-0603-25V-5%
- added D2: 3A/40V/500mV, SparkFun-DiscreteSemi:DIODE-SCHOTTKY-B340A
- added FB1, FB2, FB3, FB4, FB5, FB6: (no value), capstone:FERRITE_BEAD
- added J10: SMA, capstone:SMA
- added J7, J8: select jumper, SparkFun-Connectors:CONN_03LOCK
- added JP5: JUMPER-SMT_3_2-NC_TRACE_SILK, SparkFun-Jumpers:JUMPER-SMT_3_2-NC_TRACE_SILK
- added U4: ATMEGA328P_TQFP, SparkFun-IC-Microcontroller:ATMEGA328P_TQFP
- C10: value 1mf -> 10.0uF; device SparkFun-Capacitors:1000UF-RADIAL-5MM-35V-20%-KIT -> SparkFun-Capacitors:1.0UF-1206-50V-10%
- C11: value 10uF -> 0.1uF; device SparkFun-Capacitors:10UF-1206-6.3V-20% -> SparkFun-Capacitors:2.2UF-0805-25V-(+80/-20%)
- C12: value 10uF -> 10.0uF; device SparkFun-Capacitors:10UF-1206-6.3V-20% -> SparkFun-Capacitors:1.0UF-1206-50V-10%
- C13, C7: device SparkFun-Capacitors:2.2UF-0805-25V-(+80/-20%) -> SparkFun-Capacitors:0.18UF-0603-10V-10%
- C15, C16: value 0.1uF -> 10uF; device SparkFun-Capacitors:0.18UF-0603-10V-10% -> SparkFun-Capacitors:10UF-1206-6.3V-20%
- C19: value TBD -> 0.1uF; device SparkFun-Capacitors:0.1UF-0603-25V-5% -> SparkFun-Capacitors:0.18UF-0603-10V-10%
- C2: value 10nF -> 0.1uF; device SparkFun-Capacitors:10NF-0603-50V-10% -> SparkFun-Capacitors:2.2UF-0805-25V-(+80/-20%)
- C3: value 22uF -> 1mf; device SparkFun-Capacitors:22UF-0805-6.3V-20% -> SparkFun-Capacitors:1000UF-RADIAL-5MM-35V-20%-KIT
- C4, C5: value 10.0uF -> 1mf; device SparkFun-Capacitors:1.0UF-1206-50V-10% -> SparkFun-Capacitors:1000UF-RADIAL-5MM-35V-20%-KIT
- C6: value TBD -> 10nF; device SparkFun-Capacitors:0.1UF-0603-25V-5% -> SparkFun-Capacitors:10NF-0603-50V-10%
- C8: value 1mf -> 22uF; device SparkFun-Capacitors:1000UF-RADIAL-5MM-35V-20%-KIT -> SparkFun-Capacitors:22UF-0805-6.3V-20%
- C9: value 1mf -> TBD; device SparkFun-Capacitors:1000UF-RADIAL-5MM-35V-20%-KIT -> SparkFun-Capacitors:0.1UF-0603-25V-5%
- D1: value 3A/40V/500mV -> DIODE; device SparkFun-DiscreteSemi:DIODE-SCHOTTKY-B340A -> capstone:DIODE
- J1: value power switch -> pwr_input; device SparkFun-Connectors:CONN_02 -> SparkFun-Connectors:CONN_02LOCK
- J2: value pwr_input -> power switch; device SparkFun-Connectors:CONN_02LOCK -> SparkFun-Connectors:CONN_02
- J3: value select jumper -> (none); device SparkFun-Connectors:CONN_03LOCK -> SparkFun-Connectors:CONN_02
- J4: value select jumper -> USB-B; device SparkFun-Connectors:CONN_03LOCK -> capstone:USB-B
- J6: value (none) -> A32270-ND; device SparkFun-Connectors:CONN_02 -> capstone:A32270-ND
- JP6: value JUMPER-SMT_3_2-NC_TRACE_SILK -> card detect; device SparkFun-Jumpers:JUMPER-SMT_3_2-NC_TRACE_SILK -> SparkFun-Jumpers:JUMPER-SMT_2_NO_SILK
- L2, L3: value TBD -> 68µH/±20%/1.05A; device SparkFun-Coils:INDUCTOR-0603-33NH -> SparkFun-Coils:INDUCTOR-CR75-68UH
- L5, L6: value 68µH/±20%/1.05A -> TBD; device SparkFun-Coils:INDUCTOR-CR75-68UH -> SparkFun-Coils:INDUCTOR-0603-33NH
- R1: value 100K -> 100
- R2: value 26.7k -> 100; device SparkFun-Resistors:26.7KOHM0603-1/10W-1% -> SparkFun-Resistors:100KOHM-0402-1/16W-1%
- R6: value 100 -> 100K
- R7: value 100 -> 26.7k; device SparkFun-Resistors:100KOHM-0402-1/16W-1% -> SparkFun-Resistors:26.7KOHM0603-1/10W-1%
- U2: value ATMEGA328P_TQFP -> CSRM100; device SparkFun-IC-Microcontroller:ATMEGA328P_TQFP -> capstone:CSRM100
- renumbered U$2 to U1, U$4 to U3, U$6 to U5, U$8 to J9
Connections:
- removed net N$25: U5.RX
- removed net N$26: U5.TX
- new net INTERNAL_3.3V: C15.1, IC1.3V3OUT, IC1.VCCIO
- new net N$20: C18.1, FB3.P$1, IC1.VCC
- new net N$29: C19.1, C21.1, FB4.P$2, FB6.P$1, R11.2, U5.VCC
- new net N$30: C7.1, FB1.P$2, U2.3.3V+
- new net N$31: C17.1, FB2.P$2, U4.AREF, U4.AVCC, U4.VCC@4, U4.VCC@6
- new net N$45: C20.1, FB5.P$2, J9.VDD
- net !CSRM_LED_SINK: now also U2.LED; no longer U$3.LED
- net 3.3V: now also C12.1, C13.1, FB1.P$1, FB2.P$1, FB4.P$1, FB5.P$1; no longer C14.1, C15.1, C17.1, C18.1, C20.1, C5.1, IC1.3V3OUT, IC1.VCCIO, J9.VDD, R11.2, U$3.3.3V+, U2.AREF, U2.AVCC, U2.VCC@4, U2.VCC@6, U5.VCC
- net 5V: now also C10.1, C8.1, L4.2, R6.2; no longer C3.1, C4.1, L1.2, R1.2
- net AC_PWR: now also D1.A, J1.2; no longer J2.2, U$5.A
- net ANTENNA_CONNECTOR: now also C9.1, J6.OUT, L6.1; no longer C6.1, L3.1, U$7.OUT
- net BOOT: now also C6.1; no longer C2.1
- net CSRM_EN: now also R4.1; no longer R8.1
- net CSRM_GPIO1: now also U2.GPIO1; no longer U$3.GPIO1
- net CSRM_GPIO2: now also U2.GPIO2; no longer U$3.GPIO2
- net CSRM_GPIO3: now also U2.GPIO3; no longer U$3.GPIO3
- net CSRM_OSC_OUT: now also U2.OSC; no longer U$3.OSC
- net CSRM_PPS: now also R8.2, U4.PB0(ICP); no longer R3.2, U2.PB0(ICP)
- net CSRM_RESET: now also JP5.1, U2.RESET; no longer JP6.1, U$3.RESET
- net CSRM_RX: now also J8.2, JP2.1, R2.1; no longer J4.2, JP3.1, R6.1
- net CSRM_TX: now also J7.2, JP3.1, R3.1; no longer J3.2, JP4.1, R7.1
- net EJECT_SD: now also J3.2; no longer J6.2
- net FB: now also R6.1, R7.2; no longer R1.1, R2.2
- net GND: now also C10.2, C11.2, C12.2, C14.1, C16.1, C19.2, C2.2, C21.2, C3.-, C4.-, C5.-, C8.2, D2.A, J10.P$2, J3.1, J4.GND, J4.SHIELD, J6.GND, L5.2, L6.2, R7.1, U2.GND, U4.AGND, U4.GND@3, U4.GND@5; no longer C10.-, C11.1, C12.1, C14.2, C16.2, C3.2, C4.2, C5.2, C8.-, C9.-, D1.A, J6.1, L2.2, L3.2, R2.1, U$1.GND, U$1.SHIELD, U$3.GND, U$7.GND, U2.AGND, U2.GND@3, U2.GND@5
- net GPS_ANTENNA: now also C22.2; no longer C19.2
- net GPS_CONNECTOR: now also C22.1, FB6.P$2, J10.P$1; no longer C19.1
- net GPS_SERIAL_IN: now also JP1.1, R1.1, U5.TX; no longer JP2.1, R5.1
- net GPS_SERIAL_OUT: now also JP4.1, R5.1, U5.RX; no longer JP1.1, R4.1
- net HF_SWITCH: now also C6.2, D2.C, L4.1; no longer C2.2, D1.C, L1.1
- net MISO: now also U4.PB4(MISO); no longer U2.PB4(MISO)
- net MOSI: now also U4.PB3(MOSI/OC2); no longer U2.PB3(MOSI/OC2)
- net N$1: now also JP4.2, R5.2, U2.TX1; no longer JP1.2, R4.2, U$3.TX1
- net N$13: now also JP6.1; no longer JP7.1
- net N$15: now also D1.C, L1.1; no longer L4.1, U$5.C
- net N$16: now also C3.+, L1.2, L2.1; no longer C8.+, L4.2, L5.1
- net N$17: now also C4.+, L2.2, L3.1; no longer C9.+, L5.2, L6.1
- net N$2: now also C2.1, J2.2; no longer C7.1, J1.2
- net N$21: now also C14.2, U4.PB6(XTAL1/TOSC1); no longer C12.2, U2.PB6(XTAL1/TOSC1)
- net N$22: now also C16.2, U4.PB7(XTAL2/TOSC2); no longer C11.2, U2.PB7(XTAL2/TOSC2)
- net N$27: now also U4.PD6(AIN0); no longer U2.PD6(AIN0)
- net N$3: now also R8.1, U2.PPS; no longer R3.1, U$3.PPS
- net N$4: now also JP1.2, R1.2, U2.RX1; no longer JP2.2, R5.2, U$3.RX1
- net N$5: now also JP2.2, R2.2, U2.RX2; no longer JP3.2, R6.2, U$3.RX2
- net N$6: now also JP3.2, R3.2, U2.TX2; no longer JP4.2, R7.2, U$3.TX2
- net N$7: now also C9.2, L5.1, U2.RF_IN; no longer C6.2, L2.1, U$3.RF_IN
- net N$8: now also R4.2, U2.EN; no longer R8.2, U$3.EN
- net RESET: now also C11.1, JP5.2; no longer C13.1, JP6.2
- net SCLK: now also U4.PB5(SCK); no longer U2.PB5(SCK)
- net SD_CD: now also JP6.2, U4.PD7(AIN1); no longer JP7.2, U2.PD7(AIN1)
- net SS: now also U4.PB2(SS/OC1B); no longer U2.PB2(SS/OC1B)
- net UC_RESET: now also JP5.3, U4.PC6(/RESET); no longer JP6.3, R10.1, U2.PC6(/RESET)
- net UC_RX: now also J7.1, U4.PD0(RXD); no longer J3.1, U2.PD0(RXD)
- net UC_TX: now also J8.1, U4.PD1(TXD); no longer J4.1, U2.PD1(TXD)
- net USB_DM: now also J4.D-; no longer U$1.D-
- net USB_DP: now also J4.D+; no longer U$1.D+
- net USB_RX: now also J7.3; no longer J3.3
- net USB_TX: now also J8.3; no longer J4.3
- net USB_VCC: now also FB3.P$2, J4.VBUS; no longer C16.1, IC1.VCC, U$1.VBUS
- net VIN: now also C5.+, L3.2; no longer C10.+, L6.2
Other:
- moved on the sheet: C11, C12, C13, C14, C15, C16, C17, C18, C19, C2, C6, C7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

Commit message: latest update of schematic, sent to kevin for double check
Parts:
- removed R10: 100K, SparkFun-Resistors:100KOHM-0402-1/16W-1%
- added C23: 0.1uF, SparkFun-Capacitors:0.18UF-0603-10V-10%
- J3: value (none) -> eject sd card
- R11: value 100K -> 10K
Connections:
- removed net N$19: U5.BOOTSEL
- removed net N$23: U5.RESET
- removed net N$27: U4.PD6(AIN0)
- removed net N$9: IC1.!RESET, R10.2
- net CSRM_EN: now also U4.PD5(T1)
- net EJECT_SD: now also U4.PD4(XCK/T0)
- net GND: now also IC1.!CTS, IC1.TEST, U5.BOOTSEL
- net GPS_ENABLE: now also U4.PD6(AIN0)
- net GPS_SERIAL_IN: now also U4.PD3(INT1)
- net N$10: now also C23.1, IC1.!DTR; no longer IC1.CBUS0
- net UC_RESET: now also C23.2, U5.RESET
Other:
- moved on the sheet: C10, C12, C13, FB5, J1, J3, J4, U3
